File: STM32G031/STM32G031.kicad_pcb (KiCad board)
At the start: 2 copper layers, 1 part, among them U1 STM32G031K8T3

Commit message: minimum
Parts:
- added A1: Arduino_Nano_v2.x, Module:Arduino_Nano, F.Cu at (105.0, 105.0)
- added C1: 4.7uF, Capacitor_SMD:C_0603_1608Metric, F.Cu at (150.3, 133.8)
- added C2: 100nF, Capacitor_SMD:C_0603_1608Metric, F.Cu at (150.3, 129.4)
- added C3: 100nF, Capacitor_SMD:C_0603_1608Metric, F.Cu at (193.1, 70.1)
- added CL1: 20pF, Capacitor_SMD:C_0603_1608Metric, F.Cu at (147.3, 142.7)
- added CL2: 20pF, Capacitor_SMD:C_0603_1608Metric, F.Cu at (139.0, 142.7)
- added J1: Conn_ARM_JTAG_SWD_20, Connector_PinHeader_2.54mm:PinHeader_2x10_P2.54mm_Vertical, F.Cu at (186.1, 116.2)
- added J2: Conn_ST_STDC14, Connector_PinSocket_1.27mm:PinSocket_2x07_P1.27mm_Vertical_SMD, F.Cu at (187.7, 95.1)
- added JP1: Jumper, Connector_PinHeader_2.54mm:PinHeader_1x02_P2.54mm_Vertical, F.Cu at (126.2, 135.6)
- added SW1: SW_Push, Button_Switch_THT:SW_PUSH_6mm_H5mm, F.Cu at (180.7, 67.6)
- added Y1: Crystal_GND24, Crystal:Crystal_SMD_3225-4Pin_3.2x2.5mm, F.Cu at (143.0, 135.9)
- moved U1 112.3 mm to (141.9, 122.4), turned to 135 degrees
Connections:
- U1 pad 1: Net-(U1-Pad1) -> /PB9
- U1 pad 10: Net-(U1-Pad10) -> T_VCP_RX
- U1 pad 11: Net-(U1-Pad11) -> /PA4
- U1 pad 12: Net-(U1-Pad12) -> /PA5
- U1 pad 13: Net-(U1-Pad13) -> /PA6
- U1 pad 14: Net-(U1-Pad14) -> /PA7
- U1 pad 15: Net-(U1-Pad15) -> /PB0
- U1 pad 16: Net-(U1-Pad16) -> /PB1
- U1 pad 17: Net-(U1-Pad17) -> /PB2
- U1 pad 18: Net-(U1-Pad18) -> /PA8
- U1 pad 19: Net-(U1-Pad19) -> /PA9
- U1 pad 21: Net-(U1-Pad21) -> /PA10
- U1 pad 22: Net-(U1-Pad22) -> /PA11
- U1 pad 23: Net-(U1-Pad23) -> /PA12
- U1 pad 24: Net-(U1-Pad24) -> /SWDIO
- U1 pad 25: Net-(U1-Pad25) -> /SWCLK
- U1 pad 26: Net-(U1-Pad26) -> /PA15
- U1 pad 27: Net-(U1-Pad27) -> /PB3
- U1 pad 28: Net-(U1-Pad28) -> /PB4
- U1 pad 29: Net-(U1-Pad29) -> /PB5
- U1 pad 30: Net-(U1-Pad30) -> /PB6
- U1 pad 31: Net-(U1-Pad31) -> /PB7
- U1 pad 32: Net-(U1-Pad32) -> /PB8
- U1 pad 4: Net-(U1-Pad4) -> VDD
- U1 pad 5: Net-(U1-Pad5) -> GND
- U1 pad 6: Net-(U1-Pad6) -> /NRST
- U1 pad 7: Net-(U1-Pad7) -> /PA0
- U1 pad 8: Net-(U1-Pad8) -> /PA1
- U1 pad 9: Net-(U1-Pad9) -> T_VCP_TX
Routing:
- added copper zone on F.Cu, net GND
- added copper zone on B.Cu, net VDD
Other:
- board outline added: 100 x 100 mm

Commit message: Update STM32G031.kicad_pcb
Parts:
- moved C3 58.1 mm to (137.8, 87.8)
- moved SW1 58.1 mm to (125.4, 85.3)
Routing:
- net /NRST: track 0.00 -> 192.2 mm, vias 0 -> 2
- net /SWCLK: track 0.00 -> 87.8 mm, vias 0 -> 2
- net /SWDIO: track 0.00 -> 83.8 mm, vias 0 -> 2
- net /PB0: track 0.00 -> 71.3 mm, vias 0 -> 2
- net /PB7: track 0.00 -> 68.7 mm, vias 0 -> 1
- net /PB1: track 0.00 -> 68.4 mm, vias 0 -> 2
- net /PB9: track 0.00 -> 63.5 mm
- net /PB3: track 0.00 -> 62.8 mm, vias 0 -> 2
- net /PB6: track 0.00 -> 52.9 mm, vias 0 -> 3
- net T_VCP_TX: track 0.00 -> 52.1 mm
- net GND: track 0.00 -> 51.0 mm
- net /PA7: track 0.00 -> 49.3 mm, vias 0 -> 2
- net T_VCP_RX: track 0.00 -> 48.7 mm
- net VDD: track 0.00 -> 48.4 mm, vias 0 -> 2
- net /PA6: track 0.00 -> 47.8 mm, vias 0 -> 2
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