File: STM32G031V2/Toiletlock-V2.kicad_pcb (KiCad board)
At the start: 2 copper layers, 100 x 100 mm, 33 parts, among them J1 Conn_ST_STDC14, J2 Conn_01x02_Male, J3 Conn_ARM_JTAG_SWD_20, SW1 SW_Push, U1 STM32G031K8T3, U2 DRV8837C, U3 APDS-9960, Y1 Crystal_GND24

Commit message: add led on
Parts:
- moved RON1 58.9 mm to (136.8, 123.8)
- moved ON1 57.6 mm to (133.0, 123.8), turned to 180 degrees
Connections:
- A1 pad 17: VDD -> +3V3
- C1 pad 1: VDD -> +3V3
- C2 pad 1: VDD -> +3V3
- J1 pad 3: VDD -> +3V3
- J3 pad 1: VDD -> +3V3
- J3 pad 2: VDD -> +3V3
- JP1 pad 2: VDD -> +3V3
- U1 pad 4: VDD -> +3V3
Routing:
- net +3V3: track 0.00 -> 33.1 mm, vias 0 -> 2
- net VDD: track 24.9 -> 0.00 mm, vias 2 -> 0
- net GND: track 49.8 -> 54.2 mm
- net Net-(ON1-Pad1): track 0.00 -> 2.20 mm
- added copper zone on B.Cu, net +3V3
- removed copper zone on B.Cu, net VDD

Commit message: Finsh V2 Dev Board
Parts:
- removed BATT1: Conn_01x02_Male, Connector_JST:JST_PH_B2B-PH-K_1x02_P2.00mm_Vertical
- removed C4, C5, C6: 0.1uF, Capacitor_SMD:C_0603_1608Metric
- removed Cin1: 4.7uF, Capacitor_SMD:C_0603_1608Metric
- removed Cout1: 10uF, Capacitor_SMD:C_0603_1608Metric
- removed J2: Conn_01x02_Male, Connector_JST:JST_PH_S2B-PH-K_1x02_P2.00mm_Horizontal
- removed J3: Conn_ARM_JTAG_SWD_20, Connector_PinHeader_2.54mm:PinHeader_2x10_P2.54mm_Vertical
- removed L1: 2.2uH 2.6A, Inductor_SMD:L_Bourns-SRN4018
- removed R1, RRX1, RTX1: 22R, Resistor_SMD:R_0603_1608Metric
- removed Rfbb1: 100k, Resistor_SMD:R_0603_1608Metric
- removed Rfbt1: 453k, Resistor_SMD:R_0603_1608Metric
- removed TLV62568DBVR1: TLV62568DBV, Package_TO_SOT_SMD:SOT-23-5
- removed U2: DRV8837C, Package_SON:WSON-8-1EP_2x2mm_P0.5mm_EP0.9x1.6mm
- removed U3: APDS-9960, Silicon-Custom:APDS-9960
- removed UART1: Conn_01x04_Female, Connector_PinSocket_2.54mm:PinSocket_1x04_P2.54mm_Vertical
Other:
- board size 100 x 100 mm -> 18.5 x 46.5 mm
